File: Phylax_Version_3.kicad_pcb (KiCad board)
At the start: 2 copper layers, 60.5 x 95 mm, 59 parts, among them IC1 MCP1703AT-3302E_CB, IC2 STM32F205RET6, J2 FH19C-24S-0.5SH_10_, J4 10178589-00011LF, J6 Conn_ARM_SWD_TagConnect_TC2030, U1 SX1308, Y1 ABMM2-8.000MHZ-E2-T

Commit message: Update to version 3.3
Parts:
- removed C18, C19: 100nF X7R 0603, Capacitor_SMD:C_0603_1608Metric_Pad1.08x0.95mm_HandSolder
- removed D4, D5, D6: LED, LED_SMD:LED_0603_1608Metric_Pad1.05x0.95mm_HandSolder
- removed J4: 10178589-00011LF, 10178589-00011LF:1017858900011LF
- removed L1: SWPA4030S100MT, SWPA4030S100MT:IND-SMD_L4.0-W4.0
- removed R12: 4.7k +-1% 0603, Resistor_SMD:R_0603_1608Metric_Pad0.98x0.95mm_HandSolder
- removed R13: 1.5k +-1% 0603, Resistor_SMD:R_0603_1608Metric_Pad0.98x0.95mm_HandSolder
- removed R14: 680R +-1% 0603, Resistor_SMD:R_0603_1608Metric_Pad0.98x0.95mm_HandSolder
- removed R6: 22k +-1% 0402, Resistor_SMD:R_0402_1005Metric_Pad0.72x0.64mm_HandSolder
- removed R8: 1.5k +-1% 0402, Resistor_SMD:R_0402_1005Metric_Pad0.72x0.64mm_HandSolder
- added L2: XAL4040-103MEC, IND-SMD_L4.0-W4.0_XAL4040:IND-SMD_L4.0-W4.0_XAL4040, F.Cu at (168.8, 113.8)
- added USB1: USB4215-03-A, USB-C-SMD_GT-USB-7010B:USB-C-SMD_GT-USB-7010B, F.Cu at (164.2, 35.7)
- C15, C23: footprint Capacitor_SMD:C_0603_1608Metric_Pad1.08x0.95mm_HandSolder -> Capacitor_SMD:C_0805_2012Metric_Pad1.18x1.45mm_HandSolder
- C21: footprint Capacitor_SMD:C_0603_1608Metric_Pad1.08x0.95mm_HandSolder -> Capacitor_SMD:C_1206_3216Metric_Pad1.33x1.80mm_HandSolder
- moved C21 0.86 mm to (159.5, 108.3)
- moved R9 0.63 mm to (158.2, 77.4)
- moved C15 0.33 mm to (158.2, 75.6)
- moved C23 0.30 mm to (163.3, 118.0)
Routing:
- net +3.3V: track 122.6 -> 103.8 mm, vias 13 -> 9
- net +5V: track 97.3 -> 87.2 mm
- net VOP: track 94.6 -> 86.0 mm
- net GND: track 51.8 -> 45.3 mm, vias 1092 -> 1088
- net USB_D-: track 4.64 -> 10.5 mm, vias 0 -> 2
- net USB_D+: track 7.56 -> 10.9 mm, vias 0 -> 2
- net Net-(D6-A): track 1.59 -> 0.00 mm
- net Net-(D5-A): track 1.58 -> 0.00 mm
- net Net-(D4-A): track 1.58 -> 0.00 mm
- net IREF: track 3.82 -> 5.26 mm
- net Net-(D1-supply_voltage): track 31.8 -> 32.8 mm
- net Net-(USB1-CC2): track 2.41 -> 1.64 mm
- net SH_Right: track 6.81 -> 7.51 mm
Other:
- outline, holes or cut-outs redrawn
- board text added: "PHYLAX PCB v3.2"
- board text removed: "PHYLAX PCB v3.1"

Commit message: Update Button to be 2.55 N
Parts:
- removed S2: SKHCBEA010, SKHCBEA010:SKHCBEA010
- added S1: SKHCBGA010, SKHCBGA010:SKHCBGA010, F.Cu at (173.0, 101.0)
- S3: value SKHCBEA010 -> SKHCBGA010; footprint SKHCBEA010:SKHCBEA010 -> SKHCBGA010:SKHCBGA010
- moved S3 36.4 mm to (143.0, 101.0)
Connections:
- S3 pad 3: Net-(IC2-PC2) -> unconnected-(S3-Pad3)
- S3 pad 4: unconnected-(S3-Pad4) -> Net-(IC2-PC5)
