File: Phylax_Version_3.kicad_pcb (KiCad board)
At the start: 2 copper layers, 60.5 x 95 mm, 49 parts, among them IC1 MCP1703AT-3302E_CB, IC2 STM32F205RET6, J2 FH19C-24S-0.5SH_10_, J6 Conn_ARM_SWD_TagConnect_TC2030, U1 SX1308, Y1 ABMM2-8.000MHZ-E2-T

Commit message: Update BOM
Parts:
- C10, C11, C12, C17, C20, C4, C8, C9: value 100nF X7R 0603 -> 100nF X7R 25V 0603
Changed lines of the file:
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@@
 			)
 		)
-		(property "Value" "100nF X7R 0603"
+		(property "Value" "100nF X7R 25V 0603"
 			(at 0 1.43 90)
 			(layer "F.Fab")
@@
 			)
 		)
-		(property "Value" "100nF X7R 0603"
+		(property "Value" "100nF X7R 25V 0603"
 			(at 0 1.43 0)
 			(layer "F.Fab")
@@
 			)
 		)
-		(property "Value" "100nF X7R 0603"
+		(property "Value" "100nF X7R 25V 0603"
 			(at 0 1.43 90)
 			(layer "F.Fab")
@@
 			)
 		)
-		(property "Value" "100nF X7R 0603"
+		(property "Value" "100nF X7R 25V 0603"
 			(at 0 1.43 0)
 			(layer "F.Fab")
@@
 			)
 		)
-		(property "Value" "100nF X7R 0603"
+		(property "Value" "100nF X7R 25V 0603"
 			(at 0 1.43 0)
 			(layer "F.Fab")
@@
 			)
 		)
-		(property "LCSC Part #" "C137672"
+		(property "LCSC Part #" "C23263"
 			(at 0 0 0)
 			(unlocked yes)
@@
 			)
 		)
-		(property "Value" "100nF X7R 0603"
+		(property "Value" "100nF X7R 25V 0603"
 			(at 0 1.43 0)
 			(layer "F.Fab")
@@
 			)
 		)
-		(property "Value" "100nF X7R 0603"
+		(property "Value" "100nF X7R 25V 0603"
 			(at 0 1.43 90)
 			(layer "F.Fab")
@@
 			)
 		)
-		(property "Value" "100nF X7R 0603"
+		(property "Value" "100nF X7R 25V 0603"
 			(at 0 1.43 0)
 			(layer "F.Fab")
