File: Phylax_Version_3.kicad_sch (KiCad schematic)
At the start: 58 parts, among them IC1 MCP1703AT-3302E_CB, IC2 STM32F205RET6, J2 FH19C-24S-0.5SH_10_, J4 10178589-00011LF, J6 Conn_ARM_SWD_TagConnect_TC2030, U1 SX1308, Y1 ABMM2-8.000MHZ-E2-T

Commit message: Update to version 3.3
Parts:
- removed C18, C19: 100nF X7R 0603, Capacitor_SMD:C_0603_1608Metric_Pad1.08x0.95mm_HandSolder, symbol Device:C
- removed D4, D5, D6: LED, LED_SMD:LED_0603_1608Metric_Pad1.05x0.95mm_HandSolder, symbol Device:LED
- removed J4: 10178589-00011LF, 10178589-00011LF:1017858900011LF, symbol 10178589-00011LF:10178589-00011LF
- removed L1: SWPA4030S100MT, SWPA4030S100MT:IND-SMD_L4.0-W4.0, symbol SWPA4030S100MT:SWPA4030S100MT
- removed R12: 4.7k +-1% 0603, Resistor_SMD:R_0603_1608Metric_Pad0.98x0.95mm_HandSolder, symbol Device:R
- removed R13: 1.5k +-1% 0603, Resistor_SMD:R_0603_1608Metric_Pad0.98x0.95mm_HandSolder, symbol Device:R
- removed R14: 680R +-1% 0603, Resistor_SMD:R_0603_1608Metric_Pad0.98x0.95mm_HandSolder, symbol Device:R
- removed R6: 22k +-1% 0402, Resistor_SMD:R_0402_1005Metric_Pad0.72x0.64mm_HandSolder, symbol Device:R
- removed R8: 1.5k +-1% 0402, Resistor_SMD:R_0402_1005Metric_Pad0.72x0.64mm_HandSolder, symbol Device:R
- added L2: XAL4040-103MEC, IND-SMD_L4.0-W4.0_XAL4040:IND-SMD_L4.0-W4.0_XAL4040, symbol IND-SMD_L4.0-W4.0_XAL4040:XAL4040-103MEC
- added USB1: USB4215-03-A, USB-C-SMD_GT-USB-7010B:USB-C-SMD_GT-USB-7010B, symbol USB-C-SMD_GT-USB-7010B:USB4215-03-A
- C15, C23: footprint Capacitor_SMD:C_0603_1608Metric_Pad1.08x0.95mm_HandSolder -> Capacitor_SMD:C_0805_2012Metric_Pad1.18x1.45mm_HandSolder
- C21: footprint Capacitor_SMD:C_0603_1608Metric_Pad1.08x0.95mm_HandSolder -> Capacitor_SMD:C_1206_3216Metric_Pad1.33x1.80mm_HandSolder
Connections:
- net +5V: now also L2.1
- net GND: now also USB1.A1B12 (GND), USB1.B1A12 (GND)
- net SH_Left: now also USB1.14 (EH), USB1.16 (EH)
- net SH_Right: now also USB1.13 (EH), USB1.15 (EH)
- net USB_D+: now also USB1.A6 (Dp1), USB1.B6 (Dp2)
- net USB_D-: now also USB1.A7 (Dn1), USB1.B7 (Dn2)
- net at D3.2 (A), U1.1 (SW): now also L2.2
- net at R2.2: now also USB1.B5 (CC2)
- net at D1.4 (supply_voltage), D2.2 (A), R7.2: now also USB1.A4B9 (VBUS), USB1.B4A9 (VBUS)
- net at R1.2: now also USB1.A5 (CC1)
- no-connect marks 48 -> 50
Other:
- note removed: "Not in JLCPCB"
- moved on the sheet: C1, R1, R2, R4, R5

Commit message: Update Button to be 2.55 N
Parts:
- removed S2, S3: SKHCBEA010, SKHCBEA010:SKHCBEA010, symbol SKHCBEA010:SKHCBEA010
- added S1, S3: SKHCBGA010, SKHCBGA010:SKHCBGA010, symbol SKHCBGA010:SKHCBGA010
Connections:
- net GND: now also S1.1, S1.2, S3.1, S3.2
- net at IC2.25 (PC5): now also S3.4
- net at IC2.10 (PC2): now also S1.3
Other:
- note added: "This is 2.55 N Force"
- note removed: "This is 1.27 N Force"

Commit message: Update JCSC part number
Parts:
- C10, C11, C12, C17, C20, C22, C4, C8, C9: LCSC Part # (none) -> C14663
- R1, R2: LCSC Part # (none) -> C852856
- R10: LCSC Part # (none) -> C2974031
- R11: LCSC Part # (none) -> C98220
- R3: LCSC Part # (none) -> C313710
- R4: LCSC Part # (none) -> C2686485
- R5: LCSC Part # (none) -> C22356470
- R7: LCSC Part # (none) -> C2909316
- R9: LCSC Part # (none) -> C137672
Changed lines of the file:
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@@
 			)
 		)
+		(property "LCSC Part #" "C14663"
+			(at 93.98 52.07 90)
+			(effects
+				(font
+					(size 1.27 1.27)
+				)
+				(hide yes)
+			)
+		)
 		(pin "1"
 		)
@@
 			)
 		)
+		(property "LCSC Part #" "C22356470"
+			(at 356.87 144.78 0)
+			(effects
+				(font
+					(size 1.27 1.27)
+				)
+				(hide yes)
+			)
+		)
 		(pin "1"
 		)
@@
 			)
 		)
+		(property "LCSC Part #" "C98220"
+			(at 231.14 194.31 0)
+			(effects
+				(font
+					(size 1.27 1.27)
+				)
+				(hide yes)
+			)
+		)
 		(pin "1"
 		)
@@
 			)
 		)
+		(property "LCSC Part #" "C14663"
+			(at 148.59 81.28 90)
+			(effects
+				(font
+					(size 1.27 1.27)
+				)
+				(hide yes)
+			)
+		)
 		(pin "1"
 		)
@@
 			)
 		)
+		(property "LCSC Part #" "C14663"
+			(at 255.27 171.45 90)
+			(effects
+				(font
+					(size 1.27 1.27)
+				)
+				(hide yes)
+			)
+		)
 		(pin "1"
 		)
@@
 			)
 		)
+		(property "LCSC Part #" "C313710"
+			(at 208.28 91.44 90)
+			(effects
+				(font
+					(size 1.27 1.27)
+				)
+				(hide yes)
+			)
+		)
 		(pin "1"
 		)
@@
 			)
 		)
+		(property "LCSC Part #" "C852856"
+			(at 359.41 99.06 90)
+			(effects
+				(font
+					(size 1.27 1.27)
+				)
+				(hide yes)
+			)
+		)
 		(pin "1"
 		)
@@
 			)
 		)
+		(property "LCSC Part #" "C14663"
+			(at 64.77 96.52 90)
+			(effects
+				(font
+					(size 1.27 1.27)
+				)
+				(hide yes)
+			)
+		)
 		(pin "1"
 		)
@@
 			)
 		)
+		(property "LCSC Part #" "C14663"
+			(at 77.47 81.28 90)
+			(effects
+				(font
+					(size 1.27 1.27)
+				)
+				(hide yes)
+			)
+		)
 		(pin "1"
 		)
@@
 			)
 		)
+		(property "LCSC Part #" "C2909316"
+			(at 248.92 91.44 0)
+			(effects
+				(font
+					(size 1.27 1.27)
+				)
+				(hide yes)
+			)
+		)
 		(pin "1"
 		)
@@
 			)
 		)
+		(property "LCSC Part #" "C14663"
+			(at 182.88 200.66 90)
+			(effects
+				(font
+					(size 1.27 1.27)
+				)
+				(hide yes)
+			)
+		)
 		(pin "1"
 		)
@@
 			)
 		)
+		(property "LCSC Part #" "C137672"
+			(at 215.9 218.44 0)
+			(effects
+				(font
+					(size 1.27 1.27)
+				)
+				(hide yes)
+			)
+		)
 		(pin "1"
 		)
@@
 			)
 		)
+		(property "LCSC Part #" "C14663"
+			(at 132.08 146.05 90)
+			(effects
+				(font
+					(size 1.27 1.27)
+				)
+				(hide yes)
+			)
+		)
 		(pin "1"
 		)
@@
 			)
 		)
+		(property "LCSC Part #" "C2686485"
+			(at 182.88 88.9 90)
+			(effects
+				(font
+					(size 1.27 1.27)
+				)
+				(hide yes)
+			)
+		)
 		(pin "1"
 		)
@@
 			)
 		)
+		(property "LCSC Part #" "C14663"
+			(at 394.97 194.31 90)
+			(effects
+				(font
+					(size 1.27 1.27)
+				)
+				(hide yes)
+			)
+		)
 		(pin "1"
 		)
@@
 			)
 		)
+		(property "LCSC Part #" "C2974031"
+			(at 231.14 171.45 0)
+			(effects
+				(font
+					(size 1.27 1.27)
+				)
+				(hide yes)
+			)
+		)
 		(pin "1"
 		)
@@
 			)
 		)
+		(property "LCSC Part #" "C14663"
+			(at 99.06 148.59 90)
+			(effects
+				(font
+					(size 1.27 1.27)
+				)
+				(hide yes)
+			)
+		)
 		(pin "1"
 		)
@@
 			(effects
 				(font
+					(size 1.27 1.27)
+				)
+				(hide yes)
+			)
+		)
+		(property "LCSC Part #" "C852856"
+			(at 359.41 83.82 90)
+			(effects
+				(font

Commit message: Update BOM
Parts:
- C10, C11, C12, C17, C20, C4, C8, C9: value 100nF X7R 0603 -> 100nF X7R 25V 0603
- R9: LCSC Part # C137672 -> C23263
Changed lines of the file:
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@@
 			)
 		)
-		(property "Value" "100nF X7R 0603"
-			(at 97.79 40.386 90)
+		(property "Value" "100nF X7R 25V 0603"
+			(at 98.044 35.814 90)
 			(effects
 				(font
@@
 			)
 		)
-		(property "Value" "100nF X7R 0603"
-			(at 157.988 76.454 90)
+		(property "Value" "100nF X7R 25V 0603"
+			(at 164.846 76.962 90)
 			(effects
 				(font
@@
 			)
 		)
-		(property "Value" "100nF X7R 0603"
+		(property "Value" "100nF X7R 25V 0603"
 			(at 73.66 100.33 90)
 			(effects
@@
 			)
 		)
-		(property "Value" "100nF X7R 0603"
-			(at 67.31 77.47 90)
+		(property "Value" "100nF X7R 25V 0603"
+			(at 62.992 77.978 90)
 			(effects
 				(font
@@
 			)
 		)
-		(property "Value" "100nF X7R 0603"
+		(property "Value" "100nF X7R 25V 0603"
 			(at 178.308 192.278 90)
 			(effects
@@
 			)
 		)
-		(property "LCSC Part #" "C137672"
+		(property "LCSC Part #" "C23263"
 			(at 215.9 218.44 0)
 			(effects
@@
 			)
 		)
-		(property "Value" "100nF X7R 0603"
-			(at 136.652 155.448 90)
+		(property "Value" "100nF X7R 25V 0603"
+			(at 136.906 159.512 90)
 			(effects
 				(font
@@
 			)
 		)
-		(property "Value" "100nF X7R 0603"
+		(property "Value" "100nF X7R 25V 0603"
 			(at 399.796 207.264 90)
 			(effects
@@
 			)
 		)
-		(property "Value" "100nF X7R 0603"
-			(at 94.996 160.528 90)
+		(property "Value" "100nF X7R 25V 0603"
+			(at 94.996 165.1 90)
 			(effects
 				(font
